File: marquee sign/LED ATtiny85.brd (EAGLE design)
At the start: 57.2 x 63.5 mm, 41 parts

Commit message: Add files via upload
Parts:
- moved U$4 12.7 mm to (34.7, 4.79)
- moved LED8 2.00 mm to (34.9, 54.6)
- moved R10 2.00 mm to (34.9, 51.3)
- moved R7 2.00 mm to (43.3, 14.8)
Routing:
- net N$11: track 6.81 -> 21.5 mm, vias 0 -> 2
- net N$10: track 175.9 -> 180.7 mm, vias 0 -> 2
- net N$2: track 77.7 -> 72.9 mm, vias 2 -> 4
- net N$14: track 3.30 -> 5.36 mm
- net N$13: track 16.2 -> 17.9 mm
- net N$1: track 202.2 -> 203.1 mm
- net N$12: track 4.98 -> 5.59 mm
